File: HW/Sensor-Node/Sensor-Node.sch (KiCad schematic (older format))
At the start: 52 parts

Commit message: complete sensor-node
Parts:
- added C15, C16, C17, C18, C19: 100nF, Capacitors_SMD:C_0805_HandSoldering, symbol C
- added D5: D_ALT, nhantt-kicad-lib:D_SMA_Standard, symbol D_ALT
- added DHT1: DHT11, nhantt-kicad-lib:DHT11, symbol DHT11
- added J6: CONN_01X04, nhantt-kicad-lib:Header-4pin-2.54, symbol CONN_01X04
- added J7, J8: CONN_01X03, nhantt-kicad-lib:Header-3pin-2.54, symbol CONN_01X03
- added R23, R24, R25: 4.7k, Resistors_SMD:R_0805_HandSoldering, symbol R
- added R26, R27, R28, R29, R30, R31: 0R, Resistors_SMD:R_0805_HandSoldering, symbol R
- C4: renamed from C?; footprint Capacitors_Tantalum_SMD:CP_Tantalum_Case-C_EIA-6032-28_Reflow -> Capacitors_SMD:C_1210_HandSoldering
- C6: renamed from C?; footprint (none) -> Capacitors_SMD:C_1210_HandSoldering
- D1, D2, D3, D4: renamed from D?; footprint (none) -> LEDs:LED_0805_HandSoldering
- IC1: renamed from IC?; footprint TSSOP-20 -> nhantt-kicad-lib:TSSOP-20_4.4x6.5mm_Pitch0.65mm
- J1, J3: renamed from J?; footprint (none) -> nhantt-kicad-lib:Header-2pin-2.54-white
- J2: renamed from J?; footprint (none) -> nhantt-kicad-lib:Domino-5.08mm_4pol
- J4, J5: renamed from J?; footprint (none) -> nhantt-kicad-lib:Header-4pin-2.54
- SW1: renamed from SW?; footprint (none) -> nhantt-kicad-lib:SW_SPST_EVPBF
- U1: renamed from U?; footprint (none) -> Housings_SOIC:SOIC-8_3.9x4.9mm_Pitch1.27mm
- gave numbers to parts that had none: 38
Connections:
- net +3V3: now also R11.1, C15.1, C16.1, C17.1, C18.1, C19.1, DHT1.1 (VCC), J6.1 (P1), J7.1 (P1), J8.1 (P1), R23.2, R24.2, R25.2, R26.1, R27.1
- net +5V: now also D5.1 (K); no longer J2.1 (P1), R11.1
- net GND: now also C15.2, C16.2, C17.2, C18.2, C19.2, DHT1.4 (GND), J6.4 (P4), J7.3 (P3), J8.3 (P3), R30.2, R31.2
- net SCL: now also J6.2 (P2), R25.1
- net SDA: now also J6.3 (P3), R24.1
- net button: now also IC1.5 (OSCIN/PA1); no longer IC1.20 (PD3/AIN4/TIM2_CH2)
- net at R18.2: now also IC1.6 (OSCOUT/PA2); no longer IC1.1 (PD4/TIM2_CH1/BEEP/UART1_CK)
- net AI0: now reaches IC1.19 (PD2/AIN3[TIM2_CH3])
- net AI0: now also R26.2, R28.1
- new net: D5.2 (A), J2.1 (P1)
- new net: J7.2 (P2), R28.2, R30.1
- new net: J8.2 (P2), R29.2, R31.1
- new net AI1: IC1.20 (PD3/AIN4/TIM2_CH2), R27.2, R29.1
- new net data: DHT1.2 (DATA), IC1.1 (PD4/TIM2_CH1/BEEP/UART1_CK), R23.1
- no-connect marks 0 -> 1
Other:
- moved on the sheet: C9, D4, R10, R18
