File: HW/Master-Node/master-node.sch (KiCad schematic (older format))
At the start: 72 parts, among them J1 CONN_01X04, J2 CONN_01X06, J3 USB_OTG, J4 CONN_01X04, J5 CONN_01X08, J6 CONN_01X04, M1 NRF24L01, Q2 C1815, U1 ASM1117, U2 MC34063, U3 MAX485, U4 STM32F103C8, U5 ESP-12, Y1 Crystal

Commit message: add footprint component
Parts:
- added C26, C27: 22pF, Capacitors_SMD:C_0805_HandSoldering, symbol C
- added C28: 100nF, Capacitors_SMD:C_0805_HandSoldering, symbol C
- added D6: LED, LEDs:LED_0805, symbol LED
- added R26, R27, R28, R29: 0R, Resistors_SMD:R_0805_HandSoldering, symbol R
- added R30: 1k, Resistors_SMD:R_0805_HandSoldering, symbol R
- added R31: 10k, Resistors_SMD:R_0805_HandSoldering, symbol R
- added SW1: SW_Push, nhantt-kicad-lib:Button-6mm-smd, symbol SW_Push
- added Y2: Crystal_GND3, nhantt-kicad-lib:Crystal_Round_Horizontal_3mm_smd, symbol Crystal_GND3
- D4: footprint (none) -> nhantt-kicad-lib:SOD-80
- J2: footprint (none) -> nhantt-kicad-lib:Header-6pin-2.54-white
- J3: footprint (none) -> nhantt-kicad-lib:USB_Micro-B
- J4, J6: footprint (none) -> nhantt-kicad-lib:Header-4pin-2.54
- J5: footprint (none) -> nhantt-kicad-lib:Pin_Header_Straight_1x08_Pitch2.54mm
- L2: footprint (none) -> Resistors_SMD:R_0805_HandSoldering
- U4: footprint st-kicad-lib:LQFP-48_7x7mm_Pitch0.5mm -> nhantt-kicad-lib:LQFP-48_7x7mm_Pitch0.5mm
- U5: footprint (none) -> nhantt-kicad-lib:ESP-12E_SMD
- Y1: footprint (none) -> nhantt-kicad-lib:Crystal_SMD_HC49-SD
Connections:
- net +3V3: now also R30.2, R31.2
- net GND: now also C26.1, C27.1, C28.2, SW1.1, Y2.3
- net I/O1: now also R26.1; no longer J2.3 (P3)
- net I/O2: now also R27.1; no longer J2.4 (P4)
- net I/O3: now also R28.1; no longer J2.5 (P5)
- net I/O4: now also R29.1; no longer J2.6 (P6)
- net OSC32I: now also C26.2, Y2.2
- net OSC32O: now also C27.2, Y2.1
- net SMART_CFG: now also C28.1, R31.1, SW1.2
- net LED_STT: now reaches U4.27 (PB14/SPI2_MISO/USART3_RTS/TIM1_CH2N)
- net LED_STT: now also D6.1 (K)
- new net: J2.3 (P3), R26.2
- new net: J2.4 (P4), R27.2
- new net: J2.5 (P5), R28.2
- new net: J2.6 (P6), R29.2
- new net: D6.2 (A), R30.1
- no-connect marks 5 -> 7
Other:
- moved on the sheet: C16, C21, C22, C23

Commit message: upload layout
Parts:
- added C29: 100nF, Capacitors_SMD:C_0805_HandSoldering, symbol C
- added R32: 10k, Resistors_SMD:R_0805_HandSoldering, symbol R
- added SW2: SW_Push, nhantt-kicad-lib:Button-6mm-smd, symbol SW_Push
Connections:
- net 485TX is gone; now on net 485_TX: R15.1
- net I2C_SCL is gone; now on net SCL: U4.42 (PB6/I2C1_SCL/TIM4_CH1)
- net I2C_SDA is gone; now on net SDA: U4.43 (PB7/I2C1_SDA/TIM4_CH2)
- net +3V3: now also R32.2
- net 485_RX: now also U4.31 (USART1_RX/TIM1_CH3/PA10); no longer U4.22 (PB11/I2C2_SDA/USART3_RX)
- net 485_TX: now also U4.30 (USART1_TX/TIM1_CH2/PA9); no longer U4.21 (PB10/I2C2_SCL/USART3_TX)
- net A: now also J1.3 (P3); no longer J1.2 (P2)
- net B: now also J1.2 (P2); no longer J1.3 (P3)
- net ESP_RX: now also U4.21 (PB10/I2C2_SCL/USART3_TX); no longer U4.30 (USART1_TX/TIM1_CH2/PA9)
- net ESP_TX: now also U4.22 (PB11/I2C2_SDA/USART3_RX); no longer U4.31 (USART1_RX/TIM1_CH3/PA10)
- net GND: now also C29.2, SW2.1
- net CFG_nRF: now reaches U4.38 (JTDI/PA15)
- net CFG_nRF: now also C29.1, R32.1, SW2.2
- no-connect marks 7 -> 6

Commit message: complete layout master node
Connections:
- net SCK is gone; now on net CLK: U4.26 (PB13/SPI2_SCK/USART3_CTS/TIM1_CH1N)
- net A: now also J1.2 (P2); no longer J1.3 (P3)
- net B: now also J1.3 (P3); no longer J1.2 (P2)
- net GND: now also J1.4 (P4); no longer J1.1 (P1)
- net USB_DIS: now also U4.2 (PC13/TAMPER_RTC); no longer U4.29 (USART1_CK/TIM1_CH1/MCO/PA8)
- net VIN: now also J1.1 (P1); no longer J1.4 (P4)
- no-connect marks 6 -> 5
